File: alien-screamer.kicad_sch (KiCad schematic)
At the start: 0 parts

Commit message: hi
Parts:
- added B1, TP1: TestPoint_2Pole, symbol Connector:TestPoint_2Pole
- added C1: 100p, symbol Device:C
- added C10: 220u, symbol Device:C_Polarized
- added C11, C7, C9: .1u, symbol Device:C
- added C12, C4: 1u, symbol Device:C
- added C13: .047u, symbol Device:C
- added C14: 10u, symbol Device:C_Polarized
- added C2, C5: 1u, symbol Device:C_Polarized
- added C3: .001u, symbol Device:C
- added C6: .01u, symbol Device:C
- added C8: 470u, symbol Device:C_Polarized
- added D1: D, symbol Device:D
- added J1: AudioJack2, symbol Connector_Audio:AudioJack2
- added LFO1: LED1, symbol Device:LED
- added Q1: 2N5457, symbol Simulation_SPICE:NJFET
- added Q2, Q3: 2N3904, Package_TO_SOT_THT:TO-92_HandSolder, symbol Transistor_BJT:2N3904
- added R1, R17, R3, R9: 10K, Resistor_THT:R_Axial_DIN0207_L6.3mm_D2.5mm_P10.16mm_Horizontal, symbol Device:R
- added R10, R12: 75K, Resistor_THT:R_Axial_DIN0207_L6.3mm_D2.5mm_P10.16mm_Horizontal, symbol Device:R
- added R11, R18, R19, R25, R28, R7: 100K, Resistor_THT:R_Axial_DIN0207_L6.3mm_D2.5mm_P10.16mm_Horizontal, symbol Device:R
- added R13, R24, R6: 100K, Potentiometer_THT:Potentiometer_Alps_RK09K_Single_Vertical, symbol Device:R_Potentiometer
- added R14: 2K, Resistor_THT:R_Axial_DIN0207_L6.3mm_D2.5mm_P10.16mm_Horizontal, symbol Device:R
- added R15: 220k, Resistor_THT:R_Axial_DIN0207_L6.3mm_D2.5mm_P10.16mm_Horizontal, symbol Device:R
- added R16, R2: 2M, Resistor_THT:R_Axial_DIN0207_L6.3mm_D2.5mm_P10.16mm_Horizontal, symbol Device:R
- added R20: 15K, Resistor_THT:R_Axial_DIN0207_L6.3mm_D2.5mm_P10.16mm_Horizontal, symbol Device:R
- added R21, R22, R23, R26: 4.7K, Resistor_THT:R_Axial_DIN0207_L6.3mm_D2.5mm_P10.16mm_Horizontal, symbol Device:R
- added R27: 10, Resistor_THT:R_Axial_DIN0207_L6.3mm_D2.5mm_P10.16mm_Horizontal, symbol Device:R
- added R4: 3K, Resistor_THT:R_Axial_DIN0207_L6.3mm_D2.5mm_P10.16mm_Horizontal, symbol Device:R
- added R5: 1M, Potentiometer_THT:Potentiometer_Alps_RK09K_Single_Vertical, symbol Device:R_Potentiometer
- added R8: 300K, Resistor_THT:R_Axial_DIN0207_L6.3mm_D2.5mm_P10.16mm_Horizontal, symbol Device:R
- added S1: SW_SPST, PROJECT_FOOTPRINTS:spdt, symbol Switch:SW_SPST
- added S2: SW_SPDT_312, PROJECT_FOOTPRINTS:spdt, symbol Switch:SW_SPDT_312
- added S3: SYNC, PROJECT_FOOTPRINTS:spdt, symbol Switch:SW_SPST
- added SW1: S4, PROJECT_FOOTPRINTS:spdt, symbol Switch:SW_SPST
- added U1: LM324, symbol Amplifier_Operational:LM324
- added U2: LM386, symbol PROJECT:LM386_cUSTOM
Connections:
- new net: C6.2, R17.1, R20.1, U1.6 (-)
- new net: C1.2, R1.1, U1.14
- new net: Q2.1 (E), Q3.1 (E), R1.2
- new net: C4.2, R12.1, R19.2, R21.1, R5.2, R5.3, S1.1 (A), S3.1 (A), U1.8
- new net: C4.1, S1.2 (B), S2.2 (C)
- new net: R4.2, R5.1
- new net: C2.1, R4.1, U1.9 (-)
- new net: C12.1, R24.2
- new net: C12.2, J1.T, R25.1
- new net: R8.1, R9.2, U1.5 (+)
- new net: D1.2 (A), R8.2, U1.7
- new net: Q2.2 (B), R10.2, R14.1, R15.1, R7.2
- new net: C1.1, Q2.3 (C), R16.1, U1.13 (-)
- new net: C3.1, Q1.1 (D), Q3.3 (C), U1.2 (-)
- new net: C5.1, R12.2, S2.3 (A)
- new net: C6.1, R28.2, S3.2 (B)
- new net: C7.1, U2.6 (V+)
- new net: R6.1, S2.1 (B)
- new net: R10.1, R13.2
- new net: B1.2, SW1.1 (A)
- new net: LFO1.2 (A), R21.2
- new net: R11.2, R18.2, R19.1, U1.10 (+)
- new net: C3.2, Q1.3 (S), R24.1, R9.1, U1.1
- new net: Q1.2 (G), R2.2, R3.1
- new net: D1.1 (K), R3.2
- new net: R6.2, R7.1
- new net: R25.2, R26.1, U2.3 (+)
- new net: C10.1, C13.1, U2.5
- new net: C14.1, U2.7 (BYPASS)
- new net: C13.2, R27.1
- new net: C10.2, TP1.2
- new net BN: B1.1, C11.2, C14.2, C2.2, C5.2, C7.2, C8.2, LFO1.1 (K), R13.1, R15.2, R18.1, R2.1, R20.2, R23.2, R24.3, R26.2, R27.2, R28.1, TP1.1, U1.11 (V-), U2.2 (-), U2.4 (GND)
- new net BP: C8.1, C9.1, R11.1, R13.3, R16.2, R17.2, R22.1, R6.3, SW1.2 (B), U1.4 (V+)
- new net GND: C11.1, C9.2, J1.S, Q3.2 (B), R14.2, R22.2, R23.1, U1.12 (+), U1.3 (+)

Commit message: commit
Parts:
- added X1, X1-1, X13, X13-1, X14, X14-1, X2, X2-1, X3, X3-1, X4, X4-1, X5, X5-1, X6, X6-1, X7, X7-1, X8, X9-1: TestPoint, TestPoint:TestPoint_THTPad_D1.0mm_Drill0.5mm, symbol Connector:TestPoint
- B1, C1, J1, TP1: footprint (none) -> TestPoint:TestPoint_2Pads_Pitch5.08mm_Drill1.3mm
- C10, C8: footprint (none) -> Capacitor_THT:CP_Radial_D10.0mm_P5.00mm
- C11, C12, C13, C14, C2, C3, C4, C5, C6, C7, C9: footprint (none) -> Capacitor_THT:C_Disc_D7.5mm_W5.0mm_P5.00mm
- D1: footprint (none) -> Diode_THT:D_DO-15_P10.16mm_Horizontal
- LFO1: footprint (none) -> LED_THT:LED_D5.0mm
- Q1: footprint (none) -> Package_TO_SOT_THT:TO-92_HandSolder
- U1: footprint (none) -> Package_DIP:DIP-14_W7.62mm_LongPads
- U2: footprint (none) -> Package_DIP:DIP-8_W7.62mm_LongPads
Connections:
- net at C4.2, R12.1, R19.2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: now also X3-1.1, X3.1
- net at R4.2, R5.1: now also X1-1.1, X1.1
- net at C12.1, R24.2: now also X13-1.1, X13.1
- net at C12.2, J1.T, R25.1: now also X8.1, X9-1.1
- net at C5.1, R12.2, S2.3 (A): now also X5-1.1, X5.1
- net at C6.1, R28.2, S3.2 (B): now also X6-1.1, X6.1
- net at R10.1, R13.2: now also X4-1.1, X4.1
- net at LFO1.2 (A), R21.2: now also X7-1.1, X7.1
- net at C3.2, Q1.3 (S), R24.1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: now also X14-1.1, X14.1
- net at R6.2, R7.1: now also X2-1.1, X2.1

Commit message: Finished PCB, experimenting with connectors - unsure if it will work but have sent off PCB design for fabrication
Parts:
- removed C4: 1u, Capacitor_THT:C_Disc_D7.5mm_W5.0mm_P5.00mm, symbol Device:C
- removed J1: AudioJack2, TestPoint:TestPoint_2Pads_Pitch5.08mm_Drill1.3mm, symbol Connector_Audio:AudioJack2
- removed LFO1: LED1, LED_THT:LED_D5.0mm, symbol Device:LED
- removed R13, R24, R6: 100K, Potentiometer_THT:Potentiometer_Alps_RK09K_Single_Vertical, symbol Device:R_Potentiometer
- removed R5: 1M, Potentiometer_THT:Potentiometer_Alps_RK09K_Single_Vertical, symbol Device:R_Potentiometer
- removed S1: SW_SPST, PROJECT_FOOTPRINTS:spdt, symbol Switch:SW_SPST
- removed S2: SW_SPDT_312, PROJECT_FOOTPRINTS:spdt, symbol Switch:SW_SPDT_312
- removed S3: SYNC, PROJECT_FOOTPRINTS:spdt, symbol Switch:SW_SPST
- removed X1, X1-1, X13, X13-1, X14, X14-1, X2, X2-1, X3, X3-1, X4, X4-1, X5, X5-1, X6, X6-1, X7, X7-1, X8, X9-1: TestPoint, TestPoint:TestPoint_THTPad_D1.0mm_Drill0.5mm, symbol Connector:TestPoint
- added C4_1: 1u, Capacitor_THT:C_Disc_D7.5mm_W5.0mm_P5.00mm, symbol Device:C
- added J2, J3: Conn_02x08_Odd_Even, PROJECT_FOOTPRINTS:IDC-Header_2x08_P2.54mm_Vertical, symbol PROJECT:Conn_02x08_Odd_Even
- added J4: AudioJack2, Connector_Audio:Jack_3.5mm_PJ320E_Horizontal, symbol Connector_Audio:AudioJack2
- added LFO2: LED1, LED_THT:LED_D5.0mm, symbol Device:LED
- added R13_1, R24_1, R6_1: 100K, Potentiometer_THT:Potentiometer_Alps_RK09K_Single_Vertical, symbol Device:R_Potentiometer
- added R5_5: 1M, Potentiometer_THT:Potentiometer_Alps_RK09K_Single_Vertical, symbol Device:R_Potentiometer
- added S1_1: SW_SPST, PROJECT_FOOTPRINTS:spdt, symbol Switch:SW_SPST
- added S2_1: SW_SPDT_312, PROJECT_FOOTPRINTS:spdt, symbol Switch:SW_SPDT_312
- added S4_1: SYNC, PROJECT_FOOTPRINTS:spdt, symbol Switch:SW_SPST
- added SW2: S3_1, PROJECT_FOOTPRINTS:spdt, symbol Switch:SW_SPST
- C1: footprint TestPoint:TestPoint_2Pads_Pitch5.08mm_Drill1.3mm -> Capacitor_THT:C_Disc_D7.5mm_W5.0mm_P5.00mm
- C12, C14, C2, C5: footprint Capacitor_THT:C_Disc_D7.5mm_W5.0mm_P5.00mm -> Capacitor_THT:CP_Radial_D4.0mm_P2.00mm
- D1: footprint Diode_THT:D_DO-15_P10.16mm_Horizontal -> Diode_THT:D_T-1_P5.08mm_Horizontal
Connections:
- net BN: now also J2.BN (Pin_10), J3.BN (Pin_10), LFO2.2 (A), R13_1.1, R24_1.3
- net BP: now also B1.2, SW1.1 (A), J2.BP (Pin_9), J3.BP (Pin_9), R13_1.3, R6_1.3, S4_1.1 (A), S4_1.2 (B)
- net GND: now also J2.GND (Pin_11)
- net X6: now reaches C6.1, R28.2
- net X6: now also J2.X6 (Pin_6), J3.X6 (Pin_6), SW2.2 (B)
- net X3: now reaches R12.1, R19.2, R21.1, U1.8
- net X3: now also C4_1.1, J2.X3 (Pin_3), J3.X3 (Pin_3), R5_5.2, R5_5.3, S1_1.2 (B), SW2.1 (A)
- net X1: now reaches R4.2
- net X1: now also J2.X1 (Pin_1), J3.X1 (Pin_1), R5_5.1
- net X13: now reaches C12.1
- net X13: now also J2.X13 (Pin_13), J3.X13 (Pin_13), R24_1.2
- net X8: now reaches C12.2, R25.1
- net X8: now also J2.X8 (Pin_8), J3.X8 (Pin_8), J4.T
- net X5: now reaches C5.1, R12.2
- net X5: now also J2.X5 (Pin_5), J3.X5 (Pin_5), S2_1.3 (A)
- net X4: now reaches R10.1
- net X4: now also J2.X4 (Pin_4), J3.X4 (Pin_4), R13_1.2
- net X14: now reaches C3.2, Q1.3 (S), R9.1, U1.1
- net X14: now also J2.X14 (Pin_14), J3.X14 (Pin_14), R24_1.1
- net X7: now reaches R21.2
- net X7: now also J2.X7 (Pin_7), J3.X7 (Pin_7), LFO2.1 (K)
- net X2: now reaches R7.1
- net X2: now also J2.X2 (Pin_2), J3.X2 (Pin_2), R6_1.2
- new net: C4_1.2, S1_1.1 (A), S2_1.1 (B)
- new net: R6_1.1, S2_1.2 (C)
- new net: J3.GND (Pin_11), J4.S
- no-connect marks 0 -> 3
